File: RX.sch (EAGLE design)
At the start: 41 parts, among them IC1 MEGA8-AI, IC2 LM358D, Q1 16M

Commit message: 21/06/2017
Parts:
- added BUZZ+, BUZZ-: (no value), wirepad:SMD2
- added R11: 1k, rcl:R-EU_M1206
- added T4: (no value), transistor-neu-to92:MMBT2222ALT1-NPN-SOT23-BEC
Connections:
- new net N$17: IC1.PD3(INT1), R11.2
- new net N$18: BUZZ-.P, T4.C
- new net N$4: R11.1, T4.B
- net +5V: now also BUZZ+.P
- net GND: now also T4.E
Changed lines of the file:
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@@
 <part name="BATHV-" library="wirepad" deviceset="SMD5" device=""/>
 <part name="BATHV+" library="wirepad" deviceset="SMD5" device=""/>
+<part name="R11" library="rcl" deviceset="R-EU_" device="M1206" value="1k"/>
+<part name="T4" library="transistor-neu-to92" deviceset="*-NPN-" device="SOT23-BEC" technology="MMBT2222ALT1"/>
+<part name="GND13" library="supply1" deviceset="GND" device=""/>
+<part name="BUZZ-" library="wirepad" deviceset="SMD2" device=""/>
+<part name="BUZZ+" library="wirepad" deviceset="SMD2" device=""/>
 </parts>
 <sheets>
@@
 <instance part="C4" gate="G$1" x="-12.7" y="73.66"/>
 <instance part="R1" gate="G$1" x="43.18" y="81.28" rot="R90"/>
-<instance part="P+3" gate="1" x="43.18" y="88.9"/>
+<instance part="P+3" gate="1" x="43.18" y="99.06"/>
 <instance part="P+4" gate="1" x="-12.7" y="78.74"/>
 <instance part="P+5" gate="1" x="38.1" y="71.12"/>
@@
 <instance part="GND5" gate="1" x="43.18" y="68.58"/>
 <instance part="LED1" gate="G$1" x="2.54" y="91.44"/>
-<instance part="P+7" gate="1" x="2.54" y="96.52"/>
+<instance part="P+7" gate="1" x="-2.54" y="99.06"/>
 <instance part="R2" gate="G$1" x="2.54" y="81.28" rot="R90"/>
 <instance part="GND6" gate="1" x="2.54" y="73.66"/>
@@
 <instance part="BATHV-" gate="1" x="114.3" y="-35.56" rot="R270"/>
 <instance part="BATHV+" gate="1" x="114.3" y="-30.48" rot="R90"/>
+<instance part="R11" gate="G$1" x="129.54" y="27.94" rot="R180"/>
+<instance part="T4" gate="G$1" x="137.16" y="27.94"/>
+<instance part="GND13" gate="1" x="139.7" y="20.32"/>
+<instance part="BUZZ-" gate="1" x="137.16" y="35.56"/>
+<instance part="BUZZ+" gate="1" x="33.02" y="88.9"/>
 </instances>
 <busses>
@@
 <wire x1="58.42" y1="106.68" x2="66.04" y2="106.68" width="0.1524" layer="91"/>
 </segment>
+<segment>
+<pinref part="T4" gate="G$1" pin="E"/>
+<pinref part="GND13" gate="1" pin="GND"/>
+</segment>
 </net>
 <net name="N$3" class="0">
@@
 <pinref part="R1" gate="G$1" pin="2"/>
 <pinref part="P+3" gate="1" pin="+5V"/>
+<wire x1="43.18" y1="96.52" x2="43.18" y2="88.9" width="0.1524" layer="91"/>
+<pinref part="BUZZ+" gate="1" pin="P"/>
+<wire x1="43.18" y1="88.9" x2="43.18" y2="86.36" width="0.1524" layer="91"/>
+<wire x1="35.56" y1="88.9" x2="43.18" y2="88.9" width="0.1524" layer="91"/>
+<junction x="43.18" y="88.9"/>
 </segment>
 <segment>
@@
 <pinref part="LED1" gate="G$1" pin="A"/>
 <pinref part="P+7" gate="1" pin="+5V"/>
+<wire x1="-2.54" y1="96.52" x2="2.54" y2="93.98" width="0.1524" layer="91"/>
 </segment>
 <segment>
@@
 </segment>
 </net>
+<net name="N$4" class="0">
+<segment>
+<pinref part="R11" gate="G$1" pin="1"/>
+<pinref part="T4" gate="G$1" pin="B"/>
+</segment>
+</net>
+<net name="N$17" class="0">
+<segment>
+<pinref part="IC1" gate="G$1" pin="PD3(INT1)"/>
+<wire x1="96.52" y1="45.72" x2="111.76" y2="45.72" width="0.1524" layer="91"/>
+<wire x1="111.76" y1="45.72" x2="111.76" y2="27.94" width="0.1524" layer="91"/>
+<pinref part="R11" gate="G$1" pin="2"/>
+<wire x1="111.76" y1="27.94" x2="124.46" y2="27.94" width="0.1524" layer="91"/>
+</segment>
+</net>
+<net name="N$18" class="0">
+<segment>
+<pinref part="T4" gate="G$1" pin="C"/>
+<pinref part="BUZZ-" gate="1" pin="P"/>
+<wire x1="139.7" y1="35.56" x2="139.7" y2="33.02" width="0.1524" layer="91"/>
+</segment>
+</net>
