File: TX.brd (EAGLE design)
At the start: 80 x 50 mm, 39 parts, among them IC1 MEGA8-AI, IC2 REG1117, Q1 16M, Q2 IRLZ44Z

Commit message: 23/05/2017
Parts:
- C4: value 10u -> (none); device rcl:140CLH-1010 -> rcl:140CLH-0810
- LED1, LED2: device led:CHIP-LED0805 -> led:LED5MM
- moved LED2 11.9 mm to (40.6, 5.08), turned to 180 degrees
- moved C6 11.2 mm to (10.7, 30.0)
- moved LED1 9.16 mm to (29.7, 5.08), turned to 0 degrees
- moved R2 6.37 mm to (19.3, 5.08), turned to 180 degrees
- moved IC2 5.61 mm to (10.9, 7.87)
- moved C4 4.83 mm to (6.35, 22.4), turned to 180 degrees
- moved C8 2.05 mm to (17.5, 19.1), turned to 270 degrees
- moved C7 2.05 mm to (17.5, 13.7), turned to 90 degrees
- moved IC1 1.02 mm to (33.8, 19.6)
- moved R3 0.28 mm to (33.9, 11.9)
Connections:
- net GND: now also LED1.K, LED2.K; no longer LED1.C, LED2.C
Routing:
- net GND: track 0.00 -> 239.4 mm, vias 0 -> 6
- net +12V: track 0.00 -> 194.7 mm, vias 0 -> 1
- net +3V3: track 0.00 -> 158.0 mm, vias 0 -> 3
- net PB3: track 0.00 -> 141.1 mm, vias 0 -> 3
- net N$15: track 0.00 -> 119.5 mm
- net PB4: track 0.00 -> 43.4 mm, vias 0 -> 3
- net RESET: track 0.00 -> 39.1 mm, vias 0 -> 3
- net PULSE: track 0.00 -> 26.4 mm
- net N$7: track 0.00 -> 16.6 mm
- net N$6: track 0.00 -> 16.5 mm
- net N$4: track 0.00 -> 12.1 mm, vias 0 -> 1
- net PB5: track 0.00 -> 9.38 mm, vias 0 -> 1
- net N$2: track 0.00 -> 7.74 mm, vias 0 -> 1
- net N$1: track 0.00 -> 6.95 mm
- net N$10: track 0.00 -> 6.58 mm
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- added copper zone on layer 1, net GND
- added copper zone on layer 16, net GND
Other:
- board text added: "SAWFISH"
- board text added: "TX"
- board text added: "V0.0.1"

Commit message: 28/05/2017
Parts:
- C4: value (none) -> 10u
Changed lines of the file:
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@@
 <element name="R12" library="rcl" package="0204/7" value="27" x="73.406" y="17.78"/>
 <element name="R13" library="rcl" package="0204/7" value="27" x="73.406" y="7.62"/>
-<element name="C4" library="rcl" package="140CLH-0810" value="" x="6.35" y="22.352" rot="R180"/>
+<element name="C4" library="rcl" package="140CLH-0810" value="10u" x="6.35" y="22.352" rot="R180"/>
 <element name="LED1" library="led" package="LED5MM" value="" x="29.718" y="5.08"/>
 <element name="LED2" library="led" package="LED5MM" value="" x="40.64" y="5.08" rot="R180"/>
@@
 <contactref element="LED5" pad="A"/>
 <contactref element="LED4" pad="A"/>
-<wire x1="4.826" y1="34.014" x2="7.366" y2="34.014" width="0.6096" layer="1"/>
+<wire x1="4.826" y1="34.014" x2="7.366" y2="34.014" width="1.016" layer="1"/>
 <wire x1="7.366" y1="34.014" x2="9.786" y2="34.014" width="0.6096" layer="1"/>
 <wire x1="9.786" y1="34.014" x2="9.906" y2="33.894" width="0.6096" layer="1"/>
@@
 <wire x1="6.35" y1="18.542" x2="6.35" y2="32.49" width="0.8128" layer="1"/>
 <wire x1="6.35" y1="32.49" x2="4.826" y2="34.014" width="0.8128" layer="1"/>
-<wire x1="11.43" y1="39.284" x2="22.352" y2="39.284" width="0.8128" layer="1"/>
+<wire x1="11.43" y1="39.284" x2="22.352" y2="39.284" width="1.016" layer="1"/>
 <wire x1="22.352" y1="39.284" x2="33.528" y2="39.284" width="0.8128" layer="1"/>
 <wire x1="63.246" y1="44.45" x2="68.961" y2="44.45" width="0.8128" layer="16"/>
@@
 <wire x1="69.088" y1="46.736" x2="69.088" y2="44.577" width="0.8128" layer="16"/>
 <wire x1="69.088" y1="44.577" x2="68.961" y2="44.45" width="0.8128" layer="16"/>
-<wire x1="11.43" y1="39.284" x2="8.169" y2="39.284" width="0.6096" layer="1"/>
-<wire x1="8.169" y1="39.284" x2="7.366" y2="38.481" width="0.6096" layer="1"/>
-<wire x1="7.366" y1="38.481" x2="7.366" y2="34.014" width="0.6096" layer="1"/>
+<wire x1="11.43" y1="39.284" x2="8.169" y2="39.284" width="1.016" layer="1"/>
+<wire x1="8.169" y1="39.284" x2="7.366" y2="38.481" width="1.016" layer="1"/>
+<wire x1="7.366" y1="38.481" x2="7.366" y2="34.014" width="1.016" layer="1"/>
 </signal>
 <signal name="N$3">

Commit message: 05/07/2017
Connections:
- new net N$14: IC1.23
Changed lines of the file:
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@@
 <via x="41.91" y="8.509" extent="1-16" drill="0.6" diameter="1.4224" shape="octagon"/>
+</signal>
+<signal name="N$14">
+<contactref element="IC1" pad="23"/>
 </signal>
 </signals>
