File: TX.sch (EAGLE design)
At the start: 39 parts, among them IC1 MEGA8-AI, IC2 REG1117, Q1 16M, Q2 IRLZ44Z

Commit message: 23/05/2017
Parts:
- C4: value 10u -> (none); device rcl:CPOL-EU140CLH-1010 -> rcl:CPOL-EU140CLH-0810
- LED1, LED2: device led:LEDCHIP-LED0805 -> led:LED5MM
Changed lines of the file:
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@@
 <part name="C2" library="rcl" deviceset="CPOL-EU" device="140CLH-1010" value="330u"/>
 <part name="C3" library="rcl" deviceset="CPOL-EU" device="140CLH-1010" value="330u"/>
-<part name="C4" library="rcl" deviceset="CPOL-EU" device="140CLH-1010" value="10u"/>
 <part name="C5" library="rcl" deviceset="C-EU" device="C0402" value="0.1u"/>
 <part name="C6" library="rcl" deviceset="C-EU" device="C0402" value="0.1u"/>
@@
 <part name="+3V4" library="supply1" deviceset="+3V3" device=""/>
 <part name="R2" library="rcl" deviceset="R-EU_" device="M1206" value="680"/>
-<part name="LED1" library="led" deviceset="LED" device="CHIP-LED0805"/>
 <part name="+3V5" library="supply1" deviceset="+3V3" device=""/>
 <part name="GND6" library="supply1" deviceset="GND" device=""/>
 <part name="R3" library="rcl" deviceset="R-EU_" device="M1206" value="680"/>
-<part name="LED2" library="led" deviceset="LED" device="CHIP-LED0805"/>
 <part name="GND7" library="supply1" deviceset="GND" device=""/>
 <part name="S1" library="switch-omron" deviceset="10-XX" device=""/>
@@
 <part name="R12" library="rcl" deviceset="R-EU_" device="0204/7" value="27"/>
 <part name="R13" library="rcl" deviceset="R-EU_" device="0204/7" value="27"/>
+<part name="C4" library="rcl" deviceset="CPOL-EU" device="140CLH-0810"/>
+<part name="LED1" library="led" deviceset="LED" device="5MM"/>
+<part name="LED2" library="led" deviceset="LED" device="5MM"/>
 </parts>
 <sheets>
@@
 <instance part="C2" gate="G$1" x="-38.1" y="66.04"/>
 <instance part="C3" gate="G$1" x="-30.48" y="66.04"/>
-<instance part="C4" gate="G$1" x="10.16" y="76.2"/>
 <instance part="C5" gate="G$1" x="-55.88" y="66.04"/>
 <instance part="C6" gate="G$1" x="20.32" y="76.2"/>
@@
 <instance part="+3V4" gate="G$1" x="45.72" y="91.44"/>
 <instance part="R2" gate="G$1" x="20.32" y="106.68" rot="R90"/>
-<instance part="LED1" gate="G$1" x="20.32" y="99.06"/>
 <instance part="+3V5" gate="G$1" x="20.32" y="114.3"/>
 <instance part="GND6" gate="1" x="20.32" y="91.44"/>
 <instance part="R3" gate="G$1" x="119.38" y="27.94" rot="R90"/>
-<instance part="LED2" gate="G$1" x="119.38" y="20.32"/>
 <instance part="GND7" gate="1" x="119.38" y="12.7"/>
 <instance part="S1" gate="1" x="7.62" y="-5.08"/>
@@
 <instance part="R12" gate="G$1" x="198.12" y="12.7" rot="R90"/>
 <instance part="R13" gate="G$1" x="205.74" y="12.7" rot="R90"/>
+<instance part="C4" gate="G$1" x="10.16" y="76.2"/>
+<instance part="LED1" gate="G$1" x="20.32" y="99.06"/>
+<instance part="LED2" gate="G$1" x="119.38" y="20.32"/>
 </instances>
 <busses>
@@
 <wire x1="10.16" y1="66.04" x2="20.32" y2="66.04" width="0.1524" layer="91"/>
 <wire x1="20.32" y1="66.04" x2="20.32" y2="71.12" width="0.1524" layer="91"/>
-<pinref part="C4" gate="G$1" pin="-"/>
 <wire x1="10.16" y1="71.12" x2="10.16" y2="66.04" width="0.1524" layer="91"/>
 <junction x="10.16" y="66.04"/>
 <pinref part="GND3" gate="1" pin="GND"/>
 <pinref part="IC2" gate="G$1" pin="GND"/>
+<pinref part="C4" gate="G$1" pin="-"/>
 </segment>
 <segment>
@@
 </segment>
 <segment>
-<pinref part="LED1" gate="G$1" pin="C"/>
-<pinref part="GND6" gate="1" pin="GND"/>
-</segment>
-<segment>
-<pinref part="LED2" gate="G$1" pin="C"/>
-<pinref part="GND7" gate="1" pin="GND"/>
-</segment>
-<segment>
 <pinref part="S1" gate="1" pin="P1"/>
 <pinref part="GND8" gate="1" pin="GND"/>
@@
 <pinref part="GND12" gate="1" pin="GND"/>
 </segment>
+<segment>
+<pinref part="GND6" gate="1" pin="GND"/>
+<pinref part="LED1" gate="G$1" pin="C"/>
+</segment>
+<segment>
+<pinref part="GND7" gate="1" pin="GND"/>
+<pinref part="LED2" gate="G$1" pin="C"/>
+</segment>
 </net>
 <net name="+3V3" class="0">
 <segment>
-<pinref part="C4" gate="G$1" pin="+"/>
 <pinref part="C6" gate="G$1" pin="1"/>
 <wire x1="10.16" y1="78.74" x2="20.32" y2="78.74" width="0.1524" layer="91"/>
@@
 <pinref part="IC2" gate="G$1" pin="VOUT"/>
 <wire x1="-2.54" y1="78.74" x2="10.16" y2="78.74" width="0.1524" layer="91"/>
+<pinref part="C4" gate="G$1" pin="+"/>
 </segment>
 <segment>
@@
 </segment>
 </net>
-<net name="N$2" class="0">
-<segment>
-<pinref part="R2" gate="G$1" pin="1"/>
-<pinref part="LED1" gate="G$1" pin="A"/>
-</segment>
-</net>
 <net name="N$3" class="0">
 <segment>
@@
 <pinref part="R3" gate="G$1" pin="2"/>
 <wire x1="93.98" y1="33.02" x2="119.38" y2="33.02" width="0.1524" layer="91"/>
-</segment>
-</net>
-<net name="N$4" class="0">
-<segment>
-<pinref part="R3" gate="G$1" pin="1"/>
-<pinref part="LED2" gate="G$1" pin="A"/>
 </segment>
 </net>
@@
 </segment>
 </net>
+<net name="N$2" class="0">
+<segment>
+<pinref part="R2" gate="G$1" pin="1"/>
+<pinref part="LED1" gate="G$1" pin="A"/>
+</segment>
+</net>
+<net name="N$4" class="0">
+<segment>
+<pinref part="R3" gate="G$1" pin="1"/>
+<pinref part="LED2" gate="G$1" pin="A"/>
+</segment>
+</net>

Commit message: 28/05/2017
Parts:
- C4: value (none) -> 10u
Changed lines of the file:
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@@
 <part name="R12" library="rcl" deviceset="R-EU_" device="0204/7" value="27"/>
 <part name="R13" library="rcl" deviceset="R-EU_" device="0204/7" value="27"/>
-<part name="C4" library="rcl" deviceset="CPOL-EU" device="140CLH-0810"/>
+<part name="C4" library="rcl" deviceset="CPOL-EU" device="140CLH-0810" value="10u"/>
 <part name="LED1" library="led" deviceset="LED" device="5MM"/>
 <part name="LED2" library="led" deviceset="LED" device="5MM"/>
@@
 <wire x1="190.5" y1="30.48" x2="198.12" y2="30.48" width="0.1524" layer="91"/>
 <wire x1="198.12" y1="30.48" x2="205.74" y2="30.48" width="0.1524" layer="91"/>
-<wire x1="205.74" y1="30.48" x2="213.36" y2="30.48" width="0.1524" layer="91"/>
-<wire x1="213.36" y1="30.48" x2="213.36" y2="25.4" width="0.1524" layer="91"/>
 <junction x="149.86" y="30.48"/>
 <pinref part="LED10" gate="G$1" pin="A"/>
 <wire x1="205.74" y1="25.4" x2="205.74" y2="30.48" width="0.1524" layer="91"/>
-<junction x="205.74" y="30.48"/>
 <pinref part="LED9" gate="G$1" pin="A"/>
 <wire x1="198.12" y1="25.4" x2="198.12" y2="30.48" width="0.1524" layer="91"/>
@@
 <wire x1="190.5" y1="2.54" x2="198.12" y2="2.54" width="0.1524" layer="91"/>
 <wire x1="198.12" y1="2.54" x2="205.74" y2="2.54" width="0.1524" layer="91"/>
-<wire x1="205.74" y1="2.54" x2="213.36" y2="2.54" width="0.1524" layer="91"/>
-<wire x1="213.36" y1="2.54" x2="213.36" y2="7.62" width="0.1524" layer="91"/>
 <wire x1="160.02" y1="7.62" x2="160.02" y2="2.54" width="0.1524" layer="91"/>
 <junction x="160.02" y="2.54"/>
@@
 <junction x="198.12" y="2.54"/>
 <wire x1="205.74" y1="7.62" x2="205.74" y2="2.54" width="0.1524" layer="91"/>
-<junction x="205.74" y="2.54"/>
 <pinref part="Q2" gate="G$1" pin="D"/>
 <wire x1="149.86" y1="2.54" x2="127" y2="2.54" width="0.1524" layer="91"/>

Commit message: 05/07/2017
Connections:
- new net N$14: IC1.PC0(ADC0)
Changed lines of the file:
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@@
+</segment>
+</net>
+<net name="N$14" class="0">
+<segment>
+<pinref part="IC1" gate="G$1" pin="PC0(ADC0)"/>
+<wire x1="93.98" y1="73.66" x2="96.52" y2="73.66" width="0.1524" layer="91"/>
 </segment>
 </net>
