File: RXV2.brd (EAGLE design)
At the start: 50 x 50 mm, 38 parts, among them IC2 LM358D, K1 G5LE

Commit message: 22/07/2017
Parts:
- removed C4: 330u/16, rcl:E2,5-6
- added C7: 330/16, rcl:E2,5-7
- C1: value 330u/16 -> 330/16; device rcl:E2,5-6 -> rcl:E2,5-7
- moved C1 0.63 mm to (14.1, 5.46)
Connections:
- net +12V: now also C7.+; no longer C4.+
- net GND: now also C7.-; no longer C4.-
Routing:
- net GND: track 185.8 -> 180.5 mm
- net +5V: track 207.7 -> 208.6 mm
- removed copper zone on layer 1, net GND
Changed lines of the file:
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@@
 <setting verticaltext="up"/>
 </settings>
-<grid distance="1" unitdist="mm" unit="mm" style="lines" multiple="1" display="no" altdistance="0.025" altunitdist="inch" altunit="inch"/>
+<grid distance="5" unitdist="mm" unit="mm" style="lines" multiple="1" display="yes" altdistance="0.025" altunitdist="inch" altunit="inch"/>
 <layers>
 <layer number="1" name="Top" color="4" fill="1" visible="yes" active="yes"/>
@@
 <element name="LED1" library="led" package="CHIPLED_0805" value="" x="13.716" y="14.478" rot="R270"/>
 <element name="C5" library="capacitor-wima" package="C2.5-2" value="104" x="14.097" y="24.511" rot="R270"/>
-<element name="C4" library="rcl" package="E2,5-6" value="330u/16" x="3.937" y="5.334" rot="R270"/>
-<element name="C1" library="rcl" package="E2,5-6" value="330u/16" x="14.732" y="5.461" rot="R270"/>
 <element name="C2" library="rcl" package="E2,5-6" value="330u/16" x="46.482" y="27.94" rot="R180"/>
 <element name="C6" library="rcl" package="E2,5-6" value="330u/16" x="14.224" y="44.069" rot="R270"/>
+<element name="C7" library="rcl" package="E2,5-7" value="330/16" x="4.5974" y="5.3256" rot="R270"/>
+<element name="C1" library="rcl" package="E2,5-7" value="330/16" x="14.097" y="5.461" rot="R270"/>
 </elements>
 <signals>
@@
 <contactref element="C5" pad="2"/>
 <wire x1="10.541" y1="23.241" x2="14.097" y2="23.241" width="0.6096" layer="16"/>
-<contactref element="C4" pad="-"/>
-<contactref element="C1" pad="-"/>
-<wire x1="14.732" y1="4.191" x2="4.064" y2="4.191" width="0.6096" layer="16"/>
-<wire x1="4.064" y1="4.191" x2="3.937" y2="4.064" width="0.6096" layer="16"/>
-<wire x1="14.732" y1="4.191" x2="10.795" y2="4.191" width="0.6096" layer="16"/>
-<wire x1="10.795" y1="4.191" x2="9.525" y2="5.461" width="0.6096" layer="16"/>
+<wire x1="10.795" y1="4.191" x2="9.652" y2="5.334" width="0.6096" layer="16"/>
+<wire x1="9.652" y1="5.334" x2="9.525" y2="5.461" width="0.6096" layer="16"/>
 <wire x1="9.525" y1="5.461" x2="9.525" y2="8.509" width="0.6096" layer="16"/>
 <contactref element="C2" pad="-"/>
@@
 <wire x1="34.163" y1="12.319" x2="35.941" y2="14.097" width="0.4064" layer="16"/>
 <wire x1="35.941" y1="14.097" x2="35.941" y2="17.018" width="0.4064" layer="16"/>
-<polygon width="0.6096" layer="1" isolate="0.6096">
-<vertex x="-2.5" y="32.5"/>
-<vertex x="-2.5" y="-2.5"/>
-<vertex x="52.5" y="-2.5"/>
-<vertex x="52.5" y="32.5"/>
-</polygon>
+<contactref element="C7" pad="-"/>
+<wire x1="4.064" y1="4.191" x2="4.3434" y2="4.191" width="0.4064" layer="16"/>
+<wire x1="4.3434" y1="4.191" x2="4.5974" y2="4.0556" width="0.4064" layer="16"/>
+<contactref element="C1" pad="-"/>
+<wire x1="10.795" y1="4.191" x2="14.097" y2="4.191" width="0.6096" layer="16"/>
+<wire x1="4.5974" y1="4.0556" x2="8.3736" y2="4.0556" width="0.6096" layer="16"/>
+<wire x1="8.3736" y1="4.0556" x2="9.652" y2="5.334" width="0.6096" layer="16"/>
 <polygon width="0.6096" layer="16" isolate="0.6096">
-<vertex x="-4" y="32"/>
-<vertex x="-4" y="-2"/>
-<vertex x="52" y="-2"/>
-<vertex x="52" y="32"/>
+<vertex x="-5" y="30"/>
+<vertex x="-5" y="0"/>
+<vertex x="50" y="0"/>
+<vertex x="50" y="30"/>
 </polygon>
 </signal>
@@
 <wire x1="9.906" y1="12.573" x2="8.404" y2="12.573" width="0.6096" layer="1"/>
 <wire x1="8.404" y1="12.573" x2="8.382" y2="12.551" width="0.6096" layer="1"/>
-<contactref element="C4" pad="+"/>
 <wire x1="5.177" y1="9.346" x2="5.177" y2="7.209" width="0.6096" layer="16"/>
 <wire x1="5.177" y1="7.209" x2="4.572" y2="6.604" width="0.6096" layer="16"/>
 <via x="5.177" y="9.346" extent="1-16" drill="0.6"/>
-<wire x1="4.572" y1="6.604" x2="3.937" y2="6.604" width="0.6096" layer="16"/>
 <wire x1="10.541" y1="20.701" x2="14.224" y2="20.701" width="0.6096" layer="16"/>
 <wire x1="14.224" y1="20.701" x2="21.463" y2="27.94" width="0.6096" layer="16"/>
@@
 <wire x1="21.463" y1="27.94" x2="21.463" y2="29.594" width="0.6096" layer="1"/>
 <wire x1="21.463" y1="29.594" x2="21.714" y2="29.845" width="0.6096" layer="1"/>
+<contactref element="C7" pad="+"/>
+<wire x1="4.572" y1="6.604" x2="4.7752" y2="6.5532" width="0.4064" layer="16"/>
+<wire x1="4.7752" y1="6.5532" x2="4.5974" y2="6.5956" width="0.4064" layer="16"/>
 </signal>
 <signal name="RESET">
@@
 <contactref element="C5" pad="1"/>
 <wire x1="10.541" y1="25.781" x2="14.097" y2="25.781" width="0.6096" layer="16"/>
-<contactref element="C1" pad="+"/>
 <via x="17.018" y="11.557" extent="1-16" drill="0.6"/>
-<wire x1="14.732" y1="6.731" x2="14.732" y2="9.271" width="0.6096" layer="16"/>
 <contactref element="C2" pad="+"/>
 <wire x1="47.752" y1="27.94" x2="47.752" y2="27.178" width="0.6096" layer="16"/>
@@
 <wire x1="49.276" y1="25.654" x2="49.276" y2="21.209" width="0.6096" layer="16"/>
 <wire x1="49.276" y1="21.209" x2="48.387" y2="20.32" width="0.6096" layer="16"/>
-<wire x1="27.432" y1="3.302" x2="27.432" y2="2.794" width="0.6096" layer="16"/>
-<wire x1="27.432" y1="2.794" x2="27.432" y2="1.397" width="0.6096" layer="16"/>
+<wire x1="27.432" y1="3.302" x2="27.432" y2="1.397" width="0.6096" layer="16"/>
 <wire x1="27.432" y1="1.397" x2="27.94" y2="0.889" width="0.6096" layer="16"/>
 <wire x1="27.94" y1="0.889" x2="45.339" y2="0.889" width="0.6096" layer="16"/>
@@
 <wire x1="17.272" y1="3.429" x2="17.272" y2="5.08" width="0.6096" layer="16"/>
 <wire x1="17.272" y1="5.08" x2="15.748" y2="6.604" width="0.6096" layer="16"/>
-<wire x1="15.748" y1="6.604" x2="14.859" y2="6.604" width="0.6096" layer="16"/>
-<wire x1="14.859" y1="6.604" x2="14.732" y2="6.731" width="0.6096" layer="16"/>
+<wire x1="15.748" y1="6.604" x2="14.224" y2="6.604" width="0.6096" layer="16"/>
 <wire x1="27.054" y1="26.416" x2="32.639" y2="26.416" width="0.6096" layer="1"/>
 <wire x1="32.639" y1="26.416" x2="34.417" y2="24.638" width="0.6096" layer="1"/>
@@
 <wire x1="23.749" y1="8.89" x2="27.432" y2="5.207" width="0.6096" layer="16"/>
 <wire x1="27.432" y1="5.207" x2="27.432" y2="3.302" width="0.6096" layer="16"/>
+<contactref element="C1" pad="+"/>
+<wire x1="14.732" y1="9.271" x2="14.732" y2="9.2456" width="0.6096" layer="16"/>
+<wire x1="14.732" y1="9.2456" x2="14.224" y2="8.7376" width="0.6096" layer="16"/>
+<wire x1="14.224" y1="8.7376" x2="14.224" y2="6.858" width="0.6096" layer="16"/>
+<wire x1="14.224" y1="6.858" x2="14.097" y2="6.731" width="0.6096" layer="16"/>
+<wire x1="14.224" y1="6.604" x2="14.097" y2="6.731" width="0.6096" layer="16"/>
 </signal>
 <signal name="N$5">
